File: kiCad-FIles/Spool_Roller/Spool_Roller.kicad_sch (KiCad schematic)
At the start: 7 parts, among them J1 RotaryEncoder, U2 TMC2209_SILENTSTEPSTICK

Commit message: gerberfiles, pcb, software
those should be the final code, pcb etc.
Parts:
- added J3: POWER KNOPF, Connector_PinSocket_2.54mm:PinSocket_1x02_P2.54mm_Vertical, symbol Connector:Conn_01x02_Socket
- added J4: Barrel_Jack_MountingPin, Connector_BarrelJack:BarrelJack_Wuerth_6941xx301002, symbol Connector:Barrel_Jack_MountingPin
- added U3: ~, Connector_PinSocket_2.54mm:PinSocket_1x03_P2.54mm_Vertical, symbol New_Library:stepdown
- GUIDE1: renamed from GUIDE; footprint (none) -> Connector_PinSocket_2.00mm:PinSocket_1x04_P2.00mm_Vertical
- J1: footprint (none) -> Connector_PinSocket_2.54mm:PinSocket_1x05_P2.54mm_Vertical
- ROLL1: renamed from ROLL; footprint (none) -> Connector_PinSocket_2.00mm:PinSocket_1x04_P2.00mm_Vertical
- SH1106_Display1: renamed from SH1106_Display; footprint (none) -> Connector_PinSocket_2.54mm:PinSocket_1x04_P2.54mm_Vertical
- U1: footprint ESP32_30pin -> Espressif:joris_esp32
Connections:
- net +12V: now also J3.2 (Pin_2), U3.1 (Vin)
- net +3.3V: now also A1.13 (~{RESET}), A1.14 (~{SLEEP}), U2.13 (SPRD), U3.3 (Vout)
- net GND: now also U1.17 (GND), U1.2 (GND), J4.2, J4.MP (MountPin), U3.2 (GND)
- net at A1.15 (STEP): now also U1.25 (GPIO19); no longer U1.24 (GPIO18)
- net at A1.16 (DIR): now also U1.24 (GPIO18); no longer U1.25 (GPIO19)
- net at A1.9 (~{ENABLE}): now also U1.3 (GPIO13)
- net at U2.10 (STEP): now also U1.22 (GPIO17); no longer U1.21 (GPIO16)
- net at U2.16 (~{EN}): now also U1.10 (GPIO32)
- net at U2.9 (DIR): now also U1.21 (GPIO16); no longer U1.22 (GPIO17)
- new net: J3.1 (Pin_1), J4.1
- no-connect marks 3 -> 19
Other:
- note removed: "1-SDA 2-SCK 3-GND 4-3v3"
