File: kiCad-FIles/Spool_Roller/Spool_Roller.kicad_pcb (KiCad board)
At the start: 2 copper layers, 117 x 71 mm, 10 parts, among them J1 RotaryEncoder, J3 POWER KNOPF, J4 Barrel_Jack_MountingPin, U2 TMC2209_SILENTSTEPSTICK

Commit message: yeee
Routing:
- net Net-(J3-Pin_1): track 20.9 -> 19.9 mm
- added copper zone on B.Cu, net GND
- removed copper zone on F.Cu, net GND
